File: pcb/clock.kicad_pcb (KiCad board)
At the start: 2 copper layers, 34.8 x 24 mm, 11 parts, among them J1 Conn_01x03_Pin, J2 Conn_01x03_Pin, J3 Conn_01x03_Pin, J4 Conn_01x03_Pin, U1 ESP32-C3-SuperMini

Commit message: pcb: remove jlc serial
Other:
- board text removed: "JLCJLCJLCJLC"
Changed lines of the file:
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@@
-		)
-	)
-	(gr_text "JLCJLCJLCJLC"
-		(at 47.15 54.03 0)
-		(layer "B.SilkS")
-		(effects
-			(font
-				(size 1 1)
-				(thickness 0.1)
-			)
-			(justify left bottom mirror)
 		)
 	)
